Commit message: final version, unfinished

File: hex_walker/urdf/hex.urdf (robot description, URDF)
Before this commit: robot walker, 43 links, 42 joints
Links:
- removed link body
- added link base_link, mass 2.8; collision mesh filename=package://hex_walker/mesh/whole_body.stl scale=1.0 1.0 1.0; visual mesh filename=package://hex_walker/mesh/whole_body.stl scale=1.0 1.0 1.0
- added link imu_link, mass 0.001; visual box size=.05 .05 .05
Joints:
- added joint imu_joint: type fixed, parent base_link, child imu_link, origin xyz=0 0 0 rpy=0 0 0
- joint cam_ll_joint: parent body -> base_link
- joint cam_lr_joint: parent body -> base_link
- joint cam_ml_joint: parent body -> base_link
- joint cam_mr_joint: parent body -> base_link
- joint cam_rl_joint: parent body -> base_link
- joint cam_rr_joint: parent body -> base_link
- joint lb_servo1: parent body -> base_link
- joint lf_servo1: parent body -> base_link
- joint lm_servo1: parent body -> base_link
- joint rb_servo1: parent body -> base_link
- joint rf_servo1: parent body -> base_link
- joint rm_servo1: parent body -> base_link
